File: pcb_v1/OpticalOdometry_Board.sch (KiCad schematic (older format))
At the start: 7 parts, among them U1 ADNS-2610

Commit message: Pcb Version_1
Parts:
- removed CONN1: CONN. to main board, Socket_Strips:Socket_Strip_Angled_1x05_Pitch2.54mm, symbol Conn_01x04_Female
- removed D2: D, Diodes_THT:D_DO-41_SOD81_P7.62mm_Horizontal, symbol D
- removed U1: ADNS-2610, symbol ADNS-2610
- added D2: LED, LEDs:LED_D3.0mm, symbol LED
- added D3: D3, Diodes_THT:D_A-405_P2.54mm_Vertical_KathodeUp, symbol D
- added MK1, MK2: Mounting_Hole, Mounting_Holes:MountingHole_2.2mm_M2_Pad, symbol Mounting_Hole
- added R2: 1000R, Resistors_THT:R_Axial_DIN0204_L3.6mm_D1.6mm_P5.08mm_Horizontal, symbol R
- added U1: u, pcb_v1:ADNS-2610, symbol ADNS-2610-RESCUE-OpticalOdometry_Board
- added u1: Conector, pcb_v1:Conection, symbol Conector
- added u2: Holder, pcb_v1:Holder, symbol Holder
- D1: footprint LEDs:LED_D3.0mm_Horizontal_O3.81mm_Z2.0mm -> LEDs:LED_D3.0mm
Connections:
- wire segments 21 -> 25
Other:
- moved on the sheet: C1, C2
