File: pcb_v1.1/OpticalOdometry_Board.bak.kicad_pcb (KiCad board)
At the start: 2 copper layers, 30 x 30 mm, 16 parts

Commit message: design fixes
Routing:
- net Net-(B1-Pad7): track 63.1 -> 69.6 mm
Changed lines of the file:
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@@
     (thickness 1.6)
     (drawings 27)
-    (tracks 40)
+    (tracks 42)
     (zones 0)
     (modules 16)
@@
     (mod_text_size 1 1)
     (mod_text_width 0.15)
-    (pad_size 1.55 1.55)
-    (pad_drill 1.02)
+    (pad_size 2.8 2.8)
+    (pad_drill 2.4)
     (pad_to_mask_clearance 0.2)
     (aux_axis_origin 0 0)
     (grid_origin 0 0.5)
-    (visible_elements FFFEF77F)
+    (visible_elements FFFEE77F)
     (pcbplotparams
       (layerselection 0x00030_80000001)
@@
     (fp_line (start -2.5 -7.25) (end -2.5 -7) (layer B.SilkS) (width 0.15))
     (fp_line (start 2.5 -7.25) (end 2.5 -7) (layer B.SilkS) (width 0.15))
-    (pad 1 thru_hole circle (at 0 12.875) (size 2.8 2.8) (drill 2.6) (layers *.Cu *.Mask))
-    (pad 2 thru_hole circle (at 0 -7.75) (size 2.8 2.8) (drill 2.6) (layers *.Cu *.Mask))
+    (pad 1 thru_hole circle (at 0 12.875) (size 2.8 2.8) (drill 2.4) (layers *.Cu *.Mask))
+    (pad 2 thru_hole circle (at 0 -7.75) (size 2.8 2.8) (drill 2.4) (layers *.Cu *.Mask))
   )
   (module Capacitors_SMD:C_0805_HandSoldering (layer F.Cu)
@@
   (gr_line (start 160 77) (end 160 79.5) (layer F.SilkS) (width 0.2))
   (gr_line (start 176 79.5) (end 176 77) (layer F.SilkS) (width 0.2))
-  (gr_text "\ngithub.com/sensaorganization" (at 168 75) (layer F.SilkS)
-    (effects (font (size 1 0.7) (thickness 0.125)))
+  (gr_text "\ngithub.com/sensaorganization" (at 181 84.5 90) (layer B.SilkS)
+    (effects (font (size 1 0.7) (thickness 0.125)) (justify mirror))
   )
   (gr_line (start 153 99.25) (end 153 71.25) (angle 90) (layer Edge.Cuts) (width 0.15))
   (gr_line (start 182 99.25) (end 154 99.25) (angle 90) (layer Edge.Cuts) (width 0.15))
   (gr_line (start 154 69.25) (end 182 69.25) (angle 90) (layer Edge.Cuts) (width 0.15))
+  (segment (start 163.6 96.7) (end 164.15 97.25) (width 0.7) (layer F.Cu) (net 1))
+  (segment (start 163.6 96) (end 163.6 96.7) (width 0.7) (layer F.Cu) (net 1))
+  (segment (start 164.15 97.25) (end 170.71 97.25) (width 0.7) (layer F.Cu) (net 1))
+  (segment (start 170.71 97.25) (end 171.96 96) (width 0.7) (layer F.Cu) (net 1))
+  (segment (start 171.9 72.5) (end 171.75 72.5) (width 0.25) (layer F.Cu) (net 2))
+  (segment (start 171.75 72.5) (end 170.75 71.5) (width 0.7) (layer F.Cu) (net 2))
+  (segment (start 165.04 71.5) (end 164.04 72.5) (width 0.7) (layer F.Cu) (net 2))
+  (segment (start 170.75 71.5) (end 165.04 71.5) (width 0.7) (layer F.Cu) (net 2))
+  (segment (start 179.25 90.85) (end 179.1 91) (width 0.7) (layer F.Cu) (net 3))
+  (segment (start 179.25 88.33) (end 179.25 90.85) (width 0.7) (layer F.Cu) (net 3))
   (via (at 156.24 76.48) (size 0.6) (drill 0.4) (layers F.Cu B.Cu) (net 4))
   (via (at 155 88.75) (size 0.6) (drill 0.4) (layers F.Cu B.Cu) (net 4))
-  (segment (start 163.6 96.7) (end 164.15 97.25) (width 0.4) (layer F.Cu) (net 1))
-  (segment (start 163.6 96) (end 163.6 96.7) (width 0.4) (layer F.Cu) (net 1))
-  (segment (start 164.15 97.25) (end 170.71 97.25) (width 0.4) (layer F.Cu) (net 1))
-  (segment (start 170.71 97.25) (end 171.96 96) (width 0.4) (layer F.Cu) (net 1))
-  (segment (start 171.9 72.5) (end 171.75 72.5) (width 0.25) (layer F.Cu) (net 2))
-  (segment (start 171.75 72.5) (end 170.75 71.5) (width 0.4) (layer F.Cu) (net 2))
-  (segment (start 165.04 71.5) (end 164.04 72.5) (width 0.4) (layer F.Cu) (net 2))
-  (segment (start 170.75 71.5) (end 165.04 71.5) (width 0.4) (layer F.Cu) (net 2))
-  (segment (start 179.25 90.85) (end 179.1 91) (width 0.25) (layer F.Cu) (net 3))
-  (segment (start 179.25 88.33) (end 179.25 90.85) (width 0.4) (layer F.Cu) (net 3))
   (segment (start 156.24 79.29) (end 156.25 79.3) (width 0.25) (layer F.Cu) (net 4))
-  (segment (start 156.24 76.48) (end 156.24 79.29) (width 0.4) (layer F.Cu) (net 4))
-  (segment (start 155 88.75) (end 155 87.25) (width 0.4) (layer F.Cu) (net 4))
+  (segment (start 156.24 76.48) (end 156.24 79.29) (width 0.7) (layer F.Cu) (net 4))
+  (segment (start 155 88.75) (end 155 87.25) (width 0.7) (layer F.Cu) (net 4))
   (segment (start 175 83.25) (end 174.5 82.75) (width 0.25) (layer F.Cu) (net 5))
-  (segment (start 179.25 83.25) (end 175 83.25) (width 0.25) (layer F.Cu) (net 5))
+  (segment (start 179.25 83.25) (end 175 83.25) (width 0.5) (layer F.Cu) (net 5))
   (segment (start 179.21 80.75) (end 179.25 80.71) (width 0.25) (layer F.Cu) (net 6))
-  (segment (start 174.5 80.75) (end 179.21 80.75) (width 0.35) (layer F.Cu) (net 6))
-  (segment (start 160 85.75) (end 161.5 85.75) (width 0.4) (layer F.Cu) (net 7))
-  (segment (start 159.5 90.5) (end 159.5 86.25) (width 0.4) (layer F.Cu) (net 7))
-  (segment (start 176.9 91) (end 160 91) (width 0.4) (layer F.Cu) (net 7))
-  (segment (start 159.5 86.25) (end 160 85.75) (width 0.4) (layer F.Cu) (net 7))
-  (segment (start 160 91) (end 159.5 90.5) (width 0.4) (layer F.Cu) (net 7))
-  (segment (start 159.75 96) (end 161.4 96) (width 0.4) (layer F.Cu) (net 7))
-  (segment (start 159.5 90.5) (end 159.5 95.75) (width 0.4) (layer F.Cu) (net 7))
-  (segment (start 159.5 95.75) (end 159.75 96) (width 0.4) (layer F.Cu) (net 7))
-  (segment (start 162.63137 85.75) (end 163.25 85.13137) (width 0.4) (layer F.Cu) (net 7))
-  (segment (start 164 76.75) (end 173.75 76.75) (width 0.4) (layer F.Cu) (net 7))
-  (segment (start 161.5 85.75) (end 162.63137 85.75) (width 0.4) (layer F.Cu) (net 7))
-  (segment (start 163.25 85.13137) (end 163.25 77.5) (width 0.4) (layer F.Cu) (net 7))
-  (segment (start 174.1 76.4) (end 174.1 72.5) (width 0.4) (layer F.Cu) (net 7))
-  (segment (start 163.25 77.5) (end 164 76.75) (width 0.4) (layer F.Cu) (net 7))
-  (segment (start 173.75 76.75) (end 174.1 76.4) (width 0.4) (layer F.Cu) (net 7))
-  (segment (start 157.3 83.7) (end 156.25 83.7) (width 0.4) (layer F.Cu) (net 7))
-  (segment (start 159.5 86.25) (end 159.5 85.9) (width 0.25) (layer F.Cu) (net 7))
-  (segment (start 159.5 85.9) (end 157.3 83.7) (width 0.4) (layer F.Cu) (net 7))
-  (segment (start 158.625 86.25) (end 159.5 86.25) (width 0.4) (layer F.Cu) (net 7))
-  (segment (start 157.625 87.25) (end 158.625 86.25) (width 0.4) (layer F.Cu) (net 7))
-  (segment (start 157.5 87.25) (end 157.625 87.25) (width 0.25) (layer F.Cu) (net 7))
+  (segment (start 174.5 80.75) (end 179.21 80.75) (width 0.5) (layer F.Cu) (net 6))
+  (segment (start 174.1 73.2) (end 172.05 75.25) (width 0.7) (layer F.Cu) (net 7))
+  (segment (start 174.1 72.5) (end 174.1 73.2) (width 0.25) (layer F.Cu) (net 7))
+  (segment (start 172.05 75.25) (end 172.05 75.95) (width 0.7) (layer F.Cu) (net 7))
+  (segment (start 172.05 75.95) (end 171.25 76.75) (width 0.7) (layer F.Cu) (net 7))
+  (segment (start 171.25 76.75) (end 159.75 76.75) (width 0.7) (layer F.Cu) (net 7))
+  (segment (start 157.5 91.4) (end 157.5 87.25) (width 0.7) (layer F.Cu) (net 7))
+  (segment (start 161.4 96) (end 161.4 95.3) (width 0.7) (layer F.Cu) (net 7))
+  (segment (start 161.4 95.3) (end 157.5 91.4) (width 0.7) (layer F.Cu) (net 7))
+  (segment (start 156.25 83.7) (end 156.25 84.4) (width 0.25) (layer F.Cu) (net 7))
+  (segment (start 159.75 76.75) (end 159.75 83) (width 0.7) (layer F.Cu) (net 7))
+  (segment (start 159.05 83.7) (end 156.25 83.7) (width 0.7) (layer F.Cu) (net 7))
+  (segment (start 159.75 83) (end 159.05 83.7) (width 0.7) (layer F.Cu) (net 7))
+  (segment (start 176.9 91) (end 159.75 91) (width 0.7) (layer F.Cu) (net 7))
+  (segment (start 159.75 91) (end 159.75 87.25) (width 0.7) (layer F.Cu) (net 7))
+  (segment (start 158.75 86.25) (end 157.5 86.25) (width 0.7) (layer F.Cu) (net 7))
+  (segment (start 159.75 87.25) (end 158.75 86.25) (width 0.7) (layer F.Cu) (net 7))
+  (segment (start 157.5 85.65) (end 157.5 86.25) (width 0.7) (layer F.Cu) (net 7))
+  (segment (start 157.5 86.25) (end 157.5 87.25) (width 0.7) (layer F.Cu) (net 7))
+  (segment (start 157.1 85.25) (end 159.75 85.25) (width 0.7) (layer F.Cu) (net 7))
+  (segment (start 157.1 85.25) (end 157.5 85.65) (width 0.7) (layer F.Cu) (net 7))
+  (segment (start 156.25 84.4) (end 157.1 85.25) (width 0.7) (layer F.Cu) (net 7))
+  (segment (start 160.25 85.75) (end 161.5 85.75) (width 0.7) (layer F.Cu) (net 7))
+  (segment (start 159.75 85.25) (end 160.25 85.75) (width 0.7) (layer F.Cu) (net 7))
   (zone (net 4) (net_name "Net-(A1-Pad2)") (layer B.Cu) (hatch edge 0.508)
     (connect_pads (clearance 0.508))
