File: pcb_v1.1/OpticalOdometry_Board.sch (KiCad schematic (older format))
At the start: 14 parts, among them u1 Holder

Commit message: design fixes
Parts:
- A1: footprint pcb_v1:Conection1 -> Pin_Headers:Pin_Header_Straight_1x04_Pitch2.54mm
Connections:
- net labels added: GND, VCC
- wire segments 40 -> 24
- no-connect marks 0 -> 4
Other:
- moved on the sheet: D2, D3, R1, R2
