File: pcb_v1.1/OpticalOdometry_Board.kicad_pcb (KiCad board)
At the start: 2 copper layers, 44.3 x 32.5 mm, 11 parts, among them J1 Conn_01x04, U1 ADNS-2610, u1 Holder

Commit message: new version
Parts:
- moved C1 1.91 mm to (251.2, 80.3)
Routing:
- net GND: track 9.01 -> 11.2 mm
- net VCC: track 77.3 -> 79.2 mm
Other:
- board text added: "5V GD DT CK"
Changed lines of the file:
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@@
   (general
     (thickness 1.6)
-    (drawings 29)
+    (drawings 30)
     (tracks 38)
     (zones 0)
@@
   )
   (setup
-    (last_trace_width 0.25)
+    (last_trace_width 1)
     (user_trace_width 0.5)
     (user_trace_width 0.8)
@@
   )
   (module Capacitors_SMD:CP_Elec_5x5.7 (layer F.Cu)
-    (at 251.206 78.351 90)
+    (at 251.206 80.256 90)
     (descr "SMT capacitor, aluminium electrolytic, 5x5.7")
     (attr smd)
@@
     (descr "JST PH series connector, B4B-PH-K (http://www.jst-mfg.com/product/pdf/eng/ePH.pdf), generated with kicad-footprint-generator")
     (tags "connector JST PH side entry")
-    (fp_text reference J1 (at 3 -2.9 270) (layer F.SilkS)
+    (fp_text reference J1 (at 9.144 0.254 270) (layer F.SilkS)
       (effects (font (size 1 1) (thickness 0.15)))
     )
@@
       (xy 0.322035 -0.914207)) (layer F.SilkS) (width 0.01))
   )
+  (gr_text "5V GD DT CK" (at 249.047 72.89 90) (layer F.SilkS)
+    (effects (font (size 1 1) (thickness 0.25)))
+  )
   (gr_circle (center 234.377294 72.502498) (end 239.522 72.255) (layer Edge.Cuts) (width 0.2))
   (gr_circle (center 218.844 86.164749) (end 220.344 86.164749) (layer Edge.Cuts) (width 0.2))
@@
   (via (at 223.774 78.224) (size 0.6) (drill 0.4) (layers F.Cu B.Cu) (net 3))
   (segment (start 221.869 78.244) (end 223.754 78.244) (width 0.5) (layer F.Cu) (net 3))
-  (segment (start 249.406 76.151) (end 248.793 75.538) (width 1) (layer F.Cu) (net 3))
-  (segment (start 251.206 76.151) (end 249.406 76.151) (width 1) (layer F.Cu) (net 3))
-  (segment (start 248.793 75.538) (end 248.793 73.906) (width 1) (layer F.Cu) (net 3))
-  (segment (start 248.475 73.588) (end 246.126 73.588) (width 1) (layer F.Cu) (net 3))
-  (segment (start 248.793 73.906) (end 248.475 73.588) (width 1) (layer F.Cu) (net 3))
+  (segment (start 249.006 78.056) (end 251.206 78.056) (width 1) (layer F.Cu) (net 3))
+  (segment (start 248.475 73.588) (end 248.793 73.906) (width 1) (layer F.Cu) (net 3))
+  (segment (start 248.793 77.843) (end 249.006 78.056) (width 1) (layer F.Cu) (net 3))
+  (segment (start 248.793 73.906) (end 248.793 77.843) (width 1) (layer F.Cu) (net 3))
+  (segment (start 246.126 73.588) (end 248.475 73.588) (width 1) (layer F.Cu) (net 3))
   (segment (start 227.942 73.922) (end 226.425 73.922) (width 0.5) (layer F.Cu) (net 4))
   (segment (start 226.425 73.922) (end 225.679 74.668) (width 0.5) (layer F.Cu) (net 4))
@@
   (segment (start 223.002 86.225) (end 243.586 86.225) (width 1) (layer F.Cu) (net 4))
   (segment (start 243.586 86.225) (end 246.126 83.685) (width 1) (layer F.Cu) (net 4))
-  (segment (start 249.238 80.383) (end 246.126 80.383) (width 1) (layer F.Cu) (net 4))
-  (segment (start 249.406 80.551) (end 249.238 80.383) (width 1) (layer F.Cu) (net 4))
-  (segment (start 251.206 80.551) (end 249.406 80.551) (width 1) (layer F.Cu) (net 4))
   (segment (start 246.126 80.383) (end 246.126 75.588) (width 1) (layer F.Cu) (net 4))
-  (segment (start 246.126 83.685) (end 246.126 80.383) (width 1) (layer F.Cu) (net 4))
-  (segment (start 251.206 79.851) (end 253.089555 77.967445) (width 1) (layer F.Cu) (net 4))
-  (segment (start 253.089555 77.967445) (end 253.089555 67.026555) (width 1) (layer F.Cu) (net 4))
-  (segment (start 251.206 80.551) (end 251.206 79.851) (width 1) (layer F.Cu) (net 4))
+  (segment (start 246.294 82.456) (end 246.126 82.288) (width 1) (layer F.Cu) (net 4))
+  (segment (start 246.126 82.288) (end 246.126 80.383) (width 1) (layer F.Cu) (net 4))
+  (segment (start 251.206 82.456) (end 246.294 82.456) (width 1) (layer F.Cu) (net 4))
+  (segment (start 246.126 83.685) (end 246.126 82.288) (width 1) (layer F.Cu) (net 4))
   (segment (start 249.893 63.83) (end 246.507 63.83) (width 1) (layer F.Cu) (net 4))
+  (segment (start 253.089555 79.872445) (end 253.089555 67.026555) (width 1) (layer F.Cu) (net 4))
+  (segment (start 251.206 81.756) (end 253.089555 79.872445) (width 1) (layer F.Cu) (net 4))
   (segment (start 253.089555 67.026555) (end 249.893 63.83) (width 1) (layer F.Cu) (net 4))
+  (segment (start 251.206 82.456) (end 251.206 81.756) (width 1) (layer F.Cu) (net 4))
   (segment (start 245.46 68.922) (end 246.126 69.588) (width 1) (layer F.Cu) (net 5))
   (segment (start 240.942 68.922) (end 245.46 68.922) (width 1) (layer F.Cu) (net 5))
